File: 5V_POWER.kicad_sch (KiCad schematic)
At the start: 8 parts

Commit message: Last commit of v1
Parts:
- added C20, C21, C22, C23, C24, C25: 22uF, Capacitor_SMD:C_0805_2012Metric, symbol Device:C_Small
- R18: footprint Resistor_SMD:R_0805_2012Metric -> (none)
Connections:
- net BB_BOOT: now also C19.1; no longer R18.1
- net GND: now also R18.1, C20.2, C21.2, C22.2, C23.2, C24.2, C25.2; no longer R15.2
- net BB_AGND: now reaches R18.2
- net BB_AGND: now also R15.2; no longer C19.1
- net at R17.1: now also R14.2, R16.2; no longer L1.1
- new net BB_VOUT: C20.1, C21.1, C22.1, C23.1, C24.1, C25.1, L1.1, R17.2
Other:
- moved on the sheet: R17
