File: USB_C_PORT_POWER.kicad_sch (KiCad schematic)
At the start: 20 parts, among them U2 STL6P3LLH6, U3 STL6P3LLH6

Commit message: Last commit of v1
Connections:
- net DISCH is gone; now on net VDD: D5.1 (K), U3.1 (S), U3.2 (S), U3.3 (S)
- net GND: now also C4.1; no longer C4.2
- net VDD: now also C3.2; no longer C3.1, C4.1, R3.1, U2.5 (D), U2.6 (D), U2.7 (D), U2.8 (D), U3.5 (D), U3.6 (D), U3.7 (D), U3.8 (D)
- net VBUS_DISCHARGE: now reaches C1.1, D2.2 (A), R1.2, R2.1
- net VBUS_EN: now reaches R3.2, R4.1, R5.1, U2.4 (G), U3.4 (G)
- net at R5.2: now also C3.1; no longer C3.2
- new net USB_BUS: C4.2, R3.1, U2.5 (D), U2.6 (D), U2.7 (D), U2.8 (D), U3.5 (D), U3.6 (D), U3.7 (D), U3.8 (D)
Other:
- moved on the sheet: C3, C4, C5, C6
