File: DasLedifier.kicad_pcb (KiCad board)
At the start: 2 copper layers, 38 parts, among them J1 USB_C_Receptacle, J2 Conn_ARM_SWD_TagConnect_TC2030, J3 MCU_DEBUG, SW1 RESET_BUTTON, U1 STUSB4500QTR, U2 STL6P3LLH6, U3 STL6P3LLH6, U4 STM32F070CBTx, U5 MRF24J40MA-I/RM

Commit message: Last commit of v1
Parts:
- removed J2: Conn_ARM_SWD_TagConnect_TC2030, Connector:Tag-Connect_TC2030-IDC-FP_2x03_P1.27mm_Vertical
- removed the R7 at (42.5, 76.7)
- removed the R7 at (79.9, 37.4)
- added C14: 22nF, Capacitor_SMD:C_0805_2012Metric, F.Cu at (52.8, 28.2)
- added C15: 0.1uF, Capacitor_SMD:C_0805_2012Metric, F.Cu at (43.7, 21.1)
- added C16: 10uF, Capacitor_SMD:C_0805_2012Metric, F.Cu at (37.1, 21.1)
- added C17: 10uF, Capacitor_SMD:C_0805_2012Metric, F.Cu at (40.4, 21.1)
- added C18: 150pF, Capacitor_SMD:C_0805_2012Metric, F.Cu at (48.5, 31.8)
- added C19: 0.1uF, Capacitor_SMD:C_0805_2012Metric, F.Cu at (49.0, 17.5)
- added C20: 22uF, Capacitor_SMD:C_0805_2012Metric, F.Cu at (58.4, 41.0)
- added C21: 22uF, Capacitor_SMD:C_0805_2012Metric, F.Cu at (58.4, 38.0)
- added C22: 22uF, Capacitor_SMD:C_0805_2012Metric, F.Cu at (58.4, 35.0)
- added C23: 22uF, Capacitor_SMD:C_0805_2012Metric, F.Cu at (58.4, 32.0)
- added C24: 22uF, Capacitor_SMD:C_0805_2012Metric, F.Cu at (58.4, 29.0)
- added C25: 22uF, Capacitor_SMD:C_0805_2012Metric, F.Cu at (58.4, 25.9)
- added D8: PD_SUCCESS, LED_SMD:LED_0805_2012Metric, F.Cu at (199.4, 20.9)
- added L1: 4.7uH, Inductor_SMD:L_10.4x10.4_H4.8, F.Cu at (55.9, 18.5)
- added R10: LED Value, Resistor_SMD:R_0805_2012Metric, F.Cu at (190.5, 26.7)
- added R11: 30.1k, Resistor_SMD:R_0805_2012Metric, F.Cu at (40.6, 27.4)
- added R12: 36.1k, Resistor_SMD:R_0805_2012Metric, F.Cu at (44.2, 27.4)
- added R13: 169k, Resistor_SMD:R_0805_2012Metric, F.Cu at (44.2, 34.8)
- added R14: 30k, Resistor_SMD:R_0805_2012Metric, F.Cu at (46.5, 34.8)
- added R15: 4.1k, Resistor_SMD:R_0805_2012Metric, F.Cu at (48.5, 28.2)
- added R16: 0k, Resistor_SMD:R_0805_2012Metric, F.Cu at (50.3, 34.8)
- added R17: ?, Resistor_SMD:R_0805_2012Metric, F.Cu at (52.8, 34.8)
- added R7: 4.7k, Resistor_SMD:R_0805_2012Metric, F.Cu at (190.5, 20.8)
- added R9: LED Value, Resistor_SMD:R_0805_2012Metric, F.Cu at (190.5, 23.7)
- added SW2: SW_Nidec_CAS-120A1, Button_Switch_SMD:Nidec_Copal_CAS-120A, F.Cu at (191.0, 51.8)
- added U6: TPS56837HRPAR, STUSB4500QTR:RPA0010A-MFG, F.Cu at (47.9, 21.1)
- D3, D4: moved to B.Cu
- D6: value D_Zener -> PWR_LED; footprint Diode_SMD:D_0805_2012Metric -> LED_SMD:LED_0805_2012Metric
- J1: footprint Connector_USB:USB_C_Receptacle_Amphenol_12401548E4-2A -> Connector_USB:USB_C_Receptacle_G-Switch_GT-USB-7010ASV
- moved D7 171.7 mm to (220.2, 57.3)
- moved D6 166.4 mm to (199.4, 17.9)
- moved R8 162.8 mm to (211.0, 58.7)
- moved U4 155.1 mm to (178.0, 36.1)
- moved C10 129.4 mm to (166.8, 68.6)
- moved C11 129.4 mm to (166.8, 71.6)
- moved C12 129.4 mm to (166.8, 74.6)
- moved C7 129.4 mm to (166.8, 59.5)
- moved C8 129.4 mm to (166.8, 62.6)
- moved C9 129.4 mm to (166.8, 65.6)
- moved C13 121.0 mm to (194.9, 17.9)
- moved J3 109.2 mm to (196.7, 33.9)
- moved SW1 107.8 mm to (178.3, 48.0)
- moved D4 72.5 mm to (14.4, 16.3), turned to 180 degrees
- moved D3 65.1 mm to (14.4, 19.6), turned to 180 degrees
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Connections:
- net Net-(D2-A) renamed /USB_C_PORT_POWER/VBUS_DISCHARGE
- net Net-(U1-DISCH) renamed /DISCH
- net Net-(U2-G) renamed /USB_C_PORT_POWER/VBUS_EN
- C3 pad 1: VDD -> Net-(C3-Pad1)
- C3 pad 2: Net-(C3-Pad2) -> VDD
- C4 pad 1: VDD -> USB_GND
- C4 pad 2: USB_GND -> /USB_C_PORT_POWER/USB_BUS
- D5 pad 1: DISCH -> VDD
- D6 pad 1: MCU_VDDA -> PWR_LED
- D6 pad 2: USB_GND -> Net-(D6-A)
- R3 pad 1: VDD -> /USB_C_PORT_POWER/USB_BUS
- R5 pad 2: Net-(C3-Pad2) -> Net-(C3-Pad1)
- R6 pad 2: DISCH -> VDD
- U2 pad 5: VDD -> /USB_C_PORT_POWER/USB_BUS
- U2 pad 6: VDD -> /USB_C_PORT_POWER/USB_BUS
- U2 pad 7: VDD -> /USB_C_PORT_POWER/USB_BUS
- U2 pad 8: VDD -> /USB_C_PORT_POWER/USB_BUS
- U3 pad 1: DISCH -> VDD
- U3 pad 2: DISCH -> VDD
- U3 pad 3: DISCH -> VDD
- U3 pad 5: VDD -> /USB_C_PORT_POWER/USB_BUS
- U3 pad 6: VDD -> /USB_C_PORT_POWER/USB_BUS
- U3 pad 7: VDD -> /USB_C_PORT_POWER/USB_BUS
- U3 pad 8: VDD -> /USB_C_PORT_POWER/USB_BUS
- U5 pad 1: USB_GND -> unconnected-(U5-GND-Pad1)
- U5 pad 11: USB_GND -> unconnected-(U5-GND-Pad11)
- U5 pad 12: USB_GND -> unconnected-(U5-GND-Pad12)
Routing:
- net BB_VOUT: track 0.00 -> 20.1 mm
- net Net-(U6-EN): track 0.00 -> 14.8 mm
- net BB_FB: track 0.00 -> 11.9 mm
- net USB_GND: track 0.00 -> 10.7 mm, vias 0 -> 42
- net Net-(U6-MODE): track 0.00 -> 7.71 mm
- net Net-(R14-Pad2): track 0.00 -> 7.62 mm
- net Net-(U6-SS): track 0.00 -> 6.81 mm
- net USB_D+: track 0.00 -> 2.97 mm, vias 0 -> 1
- net USB_D-: track 0.00 -> 2.94 mm, vias 0 -> 1
- net Net-(C18-Pad2): track 0.00 -> 2.48 mm
- net BB_BOOT: track 0.00 -> 1.79 mm
- net BB_AGND: vias 0 -> 2
- added copper zone on F.Cu, net /USB_C_PORT_POWER/USB_BUS
- added copper zone on F.Cu, net BB_AGND
- added copper zone on In1.Cu, net BB_AGND
- added copper zone on F.Cu, net BB_SW
- added copper zone on F.Cu, net BB_VOUT
- added copper zone on F.Cu, net USB_GND
- added copper zone on In2.Cu, net USB_GND
- added copper zone on F.Cu, net USB_VBUS
- added copper zone on F.Cu, net VDD
Other:
- copper layers 2 -> 4

Commit message: Progress
Parts:
- removed C11: 10nF, Capacitor_SMD:C_0805_2012Metric
- removed C12: 4.7uF, Capacitor_SMD:C_0805_2012Metric
- removed C13, C15, C19: 0.1uF, Capacitor_SMD:C_0805_2012Metric
- removed C14: 22nF, Capacitor_SMD:C_0805_2012Metric
- removed C16, C17: 10uF, Capacitor_SMD:C_0805_2012Metric
- removed C18: 150pF, Capacitor_SMD:C_0805_2012Metric
- removed C20, C21, C22, C23, C24, C25: 22uF, Capacitor_SMD:C_0805_2012Metric
- removed D1, D5: ESDA25P35, STUSB4500QTR:QFN1610_STM
- removed D2: ~, Diode_SMD:D_0805_2012Metric
- removed D3, D4: ESDA25W, STUSB4500QTR:SOT323-3L_STM
- removed D6: PWR_LED, LED_SMD:LED_0805_2012Metric
- removed D7: D_Zener, Diode_SMD:D_0805_2012Metric
- removed D8: PD_SUCCESS, LED_SMD:LED_0805_2012Metric
- removed J1: USB_C_Receptacle, Connector_USB:USB_C_Receptacle_G-Switch_GT-USB-7010ASV
- removed J3: MCU_DEBUG, Connector:Tag-Connect_TC2030-IDC-NL_2x03_P1.27mm_Vertical
- removed L1: 4.7uH, Inductor_SMD:L_10.4x10.4_H4.8
- removed R10, R9: LED Value, Resistor_SMD:R_0805_2012Metric
- removed R11: 30.1k, Resistor_SMD:R_0805_2012Metric
- removed R12: 36.1k, Resistor_SMD:R_0805_2012Metric
- removed R13: 169k, Resistor_SMD:R_0805_2012Metric
- removed R14: 30k, Resistor_SMD:R_0805_2012Metric
- removed R15: 4.1k, Resistor_SMD:R_0805_2012Metric
- removed R16: 0k, Resistor_SMD:R_0805_2012Metric
- removed R17: ?, Resistor_SMD:R_0805_2012Metric
- removed R6: 1k, Resistor_SMD:R_0805_2012Metric
- removed R8: R_Small, Resistor_SMD:R_0805_2012Metric
- removed SW1: RESET_BUTTON, Button_Switch_THT:SW_PUSH_6mm
- removed SW2: SW_Nidec_CAS-120A1, Button_Switch_SMD:Nidec_Copal_CAS-120A
- removed U5: MRF24J40MA-I/RM, STUSB4500QTR:MOD12_MRF24J40MA_MCH
- removed U6: TPS56837HRPAR, STUSB4500QTR:RPA0010A-MFG
- added L2: 4.7uH, Inductor_SMD:L_0805_2012Metric, F.Cu at (66.7, 42.4)
- C1, C5: value 1uF -> 22uF
- C10, C3, C8: value 100nF -> C_Small
- C2: value 4.7uF -> C_Small
- C4, C6: value 1uF -> C_Small
- C7, C9: value 100nF -> 22uF
- R1: value 470 -> R
- R2: value 470 -> R_Small
- R3: value 100k -> 0k
- R4: value 22k -> R_Small
- R5: value 100 -> R_Small
- R7: value 4.7k -> R_Small
- U1: value STUSB4500QTR -> PTPS55289RYQR; footprint Package_DFN_QFN:QFN-24-1EP_4x4mm_P0.5mm_EP2.7x2.7mm -> footprints:RYQ0021A-MFG
- U2: value STL6P3LLH6 -> STUSB4500QTR; footprint STUSB4500QTR:POWERFLAT_3P3X3P3_STM -> Package_DFN_QFN:QFN-24-1EP_4x4mm_P0.5mm_EP2.7x2.7mm
- U3: value STL6P3LLH6 -> STM32F070CBTx; footprint STUSB4500QTR:POWERFLAT_3P3X3P3_STM -> Package_QFP:LQFP-48_7x7mm_P0.5mm
- U4: value STM32F070CBTx -> CC2520; footprint Package_QFP:LQFP-48_7x7mm_P0.5mm -> Package_DFN_QFN:QFN-28-1EP_5x5mm_P0.5mm_EP3.35x3.35mm
- moved C10 107.7 mm to (62.2, 42.8)
- moved C7 107.7 mm to (62.2, 33.7)
- moved C8 107.7 mm to (62.2, 36.8)
- moved C9 107.7 mm to (62.2, 39.8)
- moved U4 88.7 mm to (89.5, 43.3)
- moved R7 82.9 mm to (109.7, 39.4)
- moved R5 81.1 mm to (109.7, 44.3), turned to 0 degrees
- moved U2 74.2 mm to (96.3, 42.9)
- moved U3 53.3 mm to (86.9, 25.3), turned to 0 degrees
- moved U1 43.1 mm to (61.4, 25.9), turned to 0 degrees
- moved R4 41.8 mm to (66.7, 39.6)
- moved R2 41.8 mm to (66.7, 33.7)
- moved R3 39.7 mm to (66.7, 36.6), turned to 0 degrees
- moved R1 39.1 mm to (66.7, 30.7), turned to 0 degrees
- moved C2 38.1 mm to (57.8, 33.7), turned to 0 degrees
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Connections:
- C1 pad 1: /USB_C_PORT_POWER/VBUS_DISCHARGE -> /LED_SUPPLY/ISP
- C1 pad 2: USB_GND -> GND
- C10 pad 1: USB_GND -> /LED_SUPPLY/FSW
- C10 pad 2: MCU_VDDA -> /LED_SUPPLY/AGND
- C2 pad 1: USB_VBUS -> /LED_SUPPLY/COMP
- C2 pad 2: USB_GND -> Net-(C2-Pad2)
- C3 pad 1: Net-(C3-Pad1) -> /LED_SUPPLY/BOOT1
- C3 pad 2: VDD -> /LED_SUPPLY/SW1
- C4 pad 1: USB_GND -> /LED_SUPPLY/SW2
- C4 pad 2: /USB_C_PORT_POWER/USB_BUS -> /LED_SUPPLY/BOOT2
- C5 pad 1: VREG_2V7 -> /LED_SUPPLY/ISP
- C5 pad 2: USB_GND -> GND
- C6 pad 1: USB_GND -> Net-(C2-Pad2)
- C6 pad 2: VREG_1V2 -> /LED_SUPPLY/AGND
- C7 pad 1: USB_GND -> /LED_SUPPLY/ISP
- C7 pad 2: MCU_VDDA -> GND
- C8 pad 1: USB_GND -> VCC
- C8 pad 2: MCU_VDDA -> /LED_SUPPLY/AGND
- C9 pad 1: MCU_VDDA -> /LED_SUPPLY/ISP
- C9 pad 2: USB_GND -> GND
- R1 pad 1: USB_VBUS -> /LED_SUPPLY/ISP
- R1 pad 2: /USB_C_PORT_POWER/VBUS_DISCHARGE -> VDD
- R2 pad 1: /USB_C_PORT_POWER/VBUS_DISCHARGE -> /LED_SUPPLY/COMP
- R2 pad 2: VBUS_VS_Disch -> Net-(C2-Pad2)
- R3 pad 1: /USB_C_PORT_POWER/USB_BUS -> /LED_SUPPLY/AGND
- R3 pad 2: /USB_C_PORT_POWER/VBUS_EN -> GND
- R4 pad 1: /USB_C_PORT_POWER/VBUS_EN -> /LED_SUPPLY/SYNC
- R4 pad 2: VBUS_EN_SINK -> /LED_SUPPLY/AGND
- R5 pad 1: /USB_C_PORT_POWER/VBUS_EN -> /LED_SUPPLY/CDC
- R5 pad 2: Net-(C3-Pad1) -> /LED_SUPPLY/AGND
- R7 pad 1: Net-(U5-*CS) -> VDD
- R7 pad 2: USB_GND -> Net-(U1-EN_UVLO)
- U1 pad 1: CC1 -> Net-(U1-EN_UVLO)
- U1 pad 10: USB_GND -> /LED_SUPPLY/SW2
- U1 pad 11: unconnected-(U1-ATTACH-Pad11) -> /LED_SUPPLY/ISP
- U1 pad 12: PD_ADDR0 -> /LED_SUPPLY/ISP
- U1 pad 13: PD_ADDR1 -> VDD
- U1 pad 15: unconnected-(U1-GPIO-Pad15) -> /LED_SUPPLY/COMP
- U1 pad 16: VBUS_EN_SINK -> /LED_SUPPLY/CDC
- U1 pad 17: unconnected-(U1-A_B_SIDE-Pad17) -> /LED_SUPPLY/AGND
- U1 pad 18: VBUS_VS_Disch -> VCC
- U1 pad 19: PD_ALERT -> /LED_SUPPLY/BOOT2
- U1 pad 2: CC1 -> Net-(U1-EN_UVLO)
- U1 pad 20: unconnected-(U1-POWER_OK2-Pad20) -> /LED_SUPPLY/BOOT1
- U1 pad 21: VREG_1V2 -> unconnected-(U1-EXTVCC-Pad21)
- U1 pad 3: unconnected-(U1-NC-Pad3) -> BB_SCL
- U1 pad 4: CC2 -> BB_SDA
- U1 pad 5: CC2 -> /LED_SUPPLY/SYNC
- U1 pad 6: RESET -> /LED_SUPPLY/FSW
- U1 pad 7: PD_SCL -> PD_VBUS
- U1 pad 8: PD_SDA -> /LED_SUPPLY/SW1
- U1 pad 9: /DISCH -> GND
- U2 pad 1: USB_VBUS -> unconnected-(U2-CC1DB-Pad1)
- U2 pad 2: USB_VBUS -> unconnected-(U2-CC1-Pad2)
- U2 pad 3: USB_VBUS -> unconnected-(U2-NC-Pad3)
- U2 pad 4: /USB_C_PORT_POWER/VBUS_EN -> unconnected-(U2-CC2-Pad4)
- U2 pad 5: /USB_C_PORT_POWER/USB_BUS -> unconnected-(U2-CC2DB-Pad5)
- U2 pad 6: /USB_C_PORT_POWER/USB_BUS -> unconnected-(U2-RESET-Pad6)
- U2 pad 7: /USB_C_PORT_POWER/USB_BUS -> unconnected-(U2-SCL-Pad7)
- U2 pad 8: /USB_C_PORT_POWER/USB_BUS -> unconnected-(U2-SDA-Pad8)
- U3 pad 1: VDD -> unconnected-(U3-VDD-Pad1)
- U3 pad 2: VDD -> unconnected-(U3-PC13-Pad2)
- U3 pad 3: VDD -> unconnected-(U3-PC14-Pad3)
- U3 pad 4: /USB_C_PORT_POWER/VBUS_EN -> unconnected-(U3-PC15-Pad4)
- U3 pad 5: /USB_C_PORT_POWER/USB_BUS -> unconnected-(U3-PF0-Pad5)
- U3 pad 6: /USB_C_PORT_POWER/USB_BUS -> unconnected-(U3-PF1-Pad6)
- U3 pad 7: /USB_C_PORT_POWER/USB_BUS -> unconnected-(U3-NRST-Pad7)
- U3 pad 8: /USB_C_PORT_POWER/USB_BUS -> unconnected-(U3-VSSA-Pad8)
- U4 pad 1: MCU_VDDA -> unconnected-(U4-SO-Pad1)
- U4 pad 15: ZIGBEE_SCK -> unconnected-(U4-NC-Pad15)
- U4 pad 16: ZIGBEE_SDO -> unconnected-(U4-AVDD2-Pad16)
- U4 pad 17: ZIGBEE_SDI -> unconnected-(U4-RF_P-Pad17)
- U4 pad 18: unconnected-(U4-PB0-Pad18) -> (no net)
- U4 pad 23: USB_GND -> unconnected-(U4-RBIAS-Pad23)
- U4 pad 24: MCU_VDDA -> unconnected-(U4-AVDD_GUARD-Pad24)
- U4 pad 29: ZIGBEE_INT -> unconnected-(U4-AGND-Pad29)
- U4 pad 7: RESET -> unconnected-(U4-GPIO2-Pad7)
- U4 pad 8: USB_GND -> unconnected-(U4-DVDD-Pad8)
- U4 pad 9: MCU_VDDA -> unconnected-(U4-GPIO1-Pad9)
Routing:
- net BB_VOUT: track 20.1 -> 0.00 mm
- net Net-(U6-EN): track 14.8 -> 0.00 mm
- net BB_FB: track 11.9 -> 0.00 mm
- net USB_GND: track 10.7 -> 0.00 mm, vias 42 -> 0
- net Net-(U6-MODE): track 7.71 -> 0.00 mm
- net Net-(R14-Pad2): track 7.62 -> 0.00 mm
- net Net-(U6-SS): track 6.81 -> 0.00 mm
- net USB_D+: track 2.97 -> 0.00 mm, vias 1 -> 0
- net USB_D-: track 2.94 -> 0.00 mm, vias 1 -> 0
- net Net-(C18-Pad2): track 2.48 -> 0.00 mm
- net BB_BOOT: track 1.79 -> 0.00 mm
- net BB_AGND: vias 2 -> 0
- removed copper zone on F.Cu, net /USB_C_PORT_POWER/USB_BUS
- removed copper zone on F.Cu, net BB_AGND
- removed copper zone on In1.Cu, net BB_AGND
- removed copper zone on F.Cu, net BB_SW
- removed copper zone on F.Cu, net BB_VOUT
- removed copper zone on F.Cu, net USB_GND
- removed copper zone on In2.Cu, net USB_GND
- removed copper zone on F.Cu, net USB_VBUS
- removed copper zone on F.Cu, net VDD
Other:
- copper layers 4 -> 2
